File: KICAD02/PIC32MX130_SpeakingClock20170701.sch (KiCad schematic (older format))
At the start: 53 parts, among them CN1 CN-POWER, CN2 CN-ICSP, CN3 CN-UART-FTDI-TTL-232R-3V3, CN4 LCD_I2C_AQM1602XA-RN-GBW, SW1 SW_PUSH, SW2 SW_PUSH, SW3 SW_PUSH, SW4 SW_PUSH, U1 LP2950L, U3 PIC32MX130F064B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

Commit message: amend SPI DI pin for pulling up. it needs for SD card DO. chek2
Parts:
- D2: symbol LED -> LED-RESCUE-PIC32MX130_SpeakingClock20170701
- R1, R10, R11, R12, R13, R2, R3, R4, R5, R6, R7, R8, R9: symbol R -> R-RESCUE-PIC32MX130_SpeakingClock20170701
- SP1: symbol SPEAKER -> SPEAKER-RESCUE-PIC32MX130_SpeakingClock20170701
Changed lines of the file:
@@
 EESchema Schematic File Version 2
+LIBS:PIC32MX130_SpeakingClock20170701-rescue
 LIBS:mylib20161223
 LIBS:power
@@
 $EndComp
 $Comp
-L R R6
+L R-RESCUE-PIC32MX130_SpeakingClock20170701 R6
 U 1 1 585DA131
 P 5650 2800
@@
 $EndComp
 $Comp
-L +3.3V #PWR01
+L +3.3V-RESCUE-PIC32MX130_SpeakingClock20170701 #PWR01
 U 1 1 585DB21D
 P 5650 2400
@@
 $EndComp
 $Comp
-L +3.3V #PWR02
+L +3.3V-RESCUE-PIC32MX130_SpeakingClock20170701 #PWR02
 U 1 1 585DB399
 P 6350 5150
@@
 $EndComp
 $Comp
-L +3.3V #PWR03
+L +3.3V-RESCUE-PIC32MX130_SpeakingClock20170701 #PWR03
 U 1 1 585DB4C4
 P 10250 3000
@@
 $EndComp
 $Comp
-L GND #PWR04
+L GND-RESCUE-PIC32MX130_SpeakingClock20170701 #PWR04
 U 1 1 585DB8DA
 P 5400 5150
@@
 $EndComp
 $Comp
-L GND #PWR05
+L GND-RESCUE-PIC32MX130_SpeakingClock20170701 #PWR05
 U 1 1 585DBAA7
 P 5000 2850
@@
 $EndComp
 $Comp
-L +3.3V #PWR06
+L +3.3V-RESCUE-PIC32MX130_SpeakingClock20170701 #PWR06
 U 1 1 585DBACD
 P 5150 2800
@@
 $EndComp
 $Comp
-L GND #PWR07
+L GND-RESCUE-PIC32MX130_SpeakingClock20170701 #PWR07
 U 1 1 585DBD91
 P 10250 5000
@@
 $EndComp
 $Comp
-L GND #PWR08
+L GND-RESCUE-PIC32MX130_SpeakingClock20170701 #PWR08
 U 1 1 585DBEBD
 P 10250 3400
@@
 $EndComp
 $Comp
-L GND #PWR09
+L GND-RESCUE-PIC32MX130_SpeakingClock20170701 #PWR09
 U 1 1 585DC148
 P 6450 4000
@@
 $EndComp
 $Comp
-L LED D2
+L LED-RESCUE-PIC32MX130_SpeakingClock20170701 D2
 U 1 1 585E3D37
 P 10250 6400
@@
 $EndComp
 $Comp
-L GND #PWR010
+L GND-RESCUE-PIC32MX130_SpeakingClock20170701 #PWR010
 U 1 1 585E3D94
 P 10250 6650
@@
 $EndComp
 $Comp
-L R R1
+L R-RESCUE-PIC32MX130_SpeakingClock20170701 R1
 U 1 1 585E40AD
 P 10250 5900
@@
 $EndComp
 $Comp
-L GND #PWR011
+L GND-RESCUE-PIC32MX130_SpeakingClock20170701 #PWR011
 U 1 1 586CB02F
 P 14150 4350
@@
 $EndComp
 $Comp
-L GND #PWR012
+L GND-RESCUE-PIC32MX130_SpeakingClock20170701 #PWR012
 U 1 1 586CCD41
 P 14150 5350
@@
 $EndComp
 $Comp
-L GND #PWR013
+L GND-RESCUE-PIC32MX130_SpeakingClock20170701 #PWR013
 U 1 1 586D08F6
 P 3000 8800
@@
 $EndComp
 $Comp
-L GND #PWR014
+L GND-RESCUE-PIC32MX130_SpeakingClock20170701 #PWR014
 U 1 1 586D0984
 P 3750 8800
@@
 $EndComp
 $Comp
-L GND #PWR015
+L GND-RESCUE-PIC32MX130_SpeakingClock20170701 #PWR015
 U 1 1 586D09CB
 P 2200 8800
@@
 $EndComp
 $Comp
-L GND #PWR016
+L GND-RESCUE-PIC32MX130_SpeakingClock20170701 #PWR016
 U 1 1 586D1D7D
 P 1500 8100
@@
 $EndComp
 $Comp
-L R R8
+L R-RESCUE-PIC32MX130_SpeakingClock20170701 R8
 U 1 1 589CB811
 P 10900 7400
@@
 $EndComp
 $Comp
-L GND #PWR017
+L GND-RESCUE-PIC32MX130_SpeakingClock20170701 #PWR017
 U 1 1 589CC1B6
 P 11250 7950
@@
 $EndComp
 $Comp
-L GND #PWR018
+L GND-RESCUE-PIC32MX130_SpeakingClock20170701 #PWR018
 U 1 1 589CC210
 P 11750 8600
@@
 $EndComp
 $Comp
-L SPEAKER SP1
+L SPEAKER-RESCUE-PIC32MX130_SpeakingClock20170701 SP1
 U 1 1 589D1EA3
 P 14300 8150
@@
 $EndComp
 $Comp
-L GND #PWR020
+L GND-RESCUE-PIC32MX130_SpeakingClock20170701 #PWR020
 U 1 1 589EFB56
 P 12350 8800
@@
 $EndComp
 $Comp
-L GND #PWR021
+L GND-RESCUE-PIC32MX130_SpeakingClock20170701 #PWR021
 U 1 1 589EFBBE
 P 13650 8800
@@
 $EndComp
 $Comp
-L GND #PWR022
+L GND-RESCUE-PIC32MX130_SpeakingClock20170701 #PWR022
 U 1 1 589FE7D0
 P 6350 5450
@@
 $EndComp
 $Comp
-L GND #PWR023
+L GND-RESCUE-PIC32MX130_SpeakingClock20170701 #PWR023
 U 1 1 58B3561E
 P 3600 4900
@@
 $EndComp
 $Comp
-L GND #PWR024
+L GND-RESCUE-PIC32MX130_SpeakingClock20170701 #PWR024
 U 1 1 58BC870B
 P 14150 6400
@@
 $EndComp
 $Comp
-L R R2
+L R-RESCUE-PIC32MX130_SpeakingClock20170701 R2
 U 1 1 58D90DD8
 P 6300 1300
@@
 $EndComp
 $Comp
-L R R3
+L R-RESCUE-PIC32MX130_SpeakingClock20170701 R3
 U 1 1 58D90F49
 P 6300 1850
@@
 $EndComp
 $Comp
-L GND #PWR026
+L GND-RESCUE-PIC32MX130_SpeakingClock20170701 #PWR026
 U 1 1 58D90FD6
 P 6300 2200
@@
 495 <- 1.598v <- 5v\n396 <- 1.278v <- 4v\n
 $Comp
-L R R5
+L R-RESCUE-PIC32MX130_SpeakingClock20170701 R5
 U 1 1 58DC828B
 P 12350 6800
@@
 $EndComp
 $Comp
-L +3.3V #PWR028
+L +3.3V-RESCUE-PIC32MX130_SpeakingClock20170701 #PWR028
 U 1 1 58DE9D79
 P 3750 7700
@@
 $EndComp
 $Comp
-L R R12
+L R-RESCUE-PIC32MX130_SpeakingClock20170701 R12
 U 1 1 58E319B3
 P 11450 4950
@@
 $EndComp
 $Comp
-L R R11
+L R-RESCUE-PIC32MX130_SpeakingClock20170701 R11
 U 1 1 58E31A7A
 P 11250 4950
@@
 $EndComp
 $Comp
-L R R7
+L R-RESCUE-PIC32MX130_SpeakingClock20170701 R7
 U 1 1 58EA3709
 P 6900 1850
@@
 $EndComp
 $Comp
-L GND #PWR029
+L GND-RESCUE-PIC32MX130_SpeakingClock20170701 #PWR029
 U 1 1 58EA3A16
 P 6900 2200
@@
 $EndComp
 $Comp
-L R R4
+L R-RESCUE-PIC32MX130_SpeakingClock20170701 R4
 U 1 1 58EAC1DD
 P 4150 8050
@@
 $EndComp
 $Comp
-L GND #PWR030
+L GND-RESCUE-PIC32MX130_SpeakingClock20170701 #PWR030
 U 1 1 58EAC97B
 P 4350 8800
@@
 NoConn ~ 12450 5450
 $Comp
-L R R13
+L R-RESCUE-PIC32MX130_SpeakingClock20170701 R13
 U 1 1 58F9E7DB
 P 14500 6550
@@
 $EndComp
 $Comp
-L R R9
+L R-RESCUE-PIC32MX130_SpeakingClock20170701 R9
 U 1 1 59288018
 P 6250 4850
@@
 Since FTDI cable is supplying +5V, \npin 4 is not connected
 $Comp
-L R R10
+L R-RESCUE-PIC32MX130_SpeakingClock20170701 R10
 U 1 1 592ADD50
 P 11750 7650
@@
 $EndComp
 $Comp
-L +3.3V #PWR032
+L +3.3V-RESCUE-PIC32MX130_SpeakingClock20170701 #PWR032
 U 1 1 5939C790
 P 14150 3900
@@
 NoConn ~ 14400 1000
 $Comp
-L +3.3V #PWR033
+L +3.3V-RESCUE-PIC32MX130_SpeakingClock20170701 #PWR033
 U 1 1 593C4983
 P 6900 950
@@
 $EndComp
 $Comp
-L +3.3V #PWR034
+L +3.3V-RESCUE-PIC32MX130_SpeakingClock20170701 #PWR034
 U 1 1 594AA504
 P 14050 2400
@@
 $EndComp
 $Comp
-L GND #PWR035
+L GND-RESCUE-PIC32MX130_SpeakingClock20170701 #PWR035
 U 1 1 594AA5A8
 P 14050 2850
